Commit message: fix some errors

File: fetch_description/urdf/fetch_inertial.xacro (robot description, xacro)
@@ -112,5 +112,5 @@
         <origin xyz="-0.01 0 0" rpy="${mesh_offset_rpy}"/>
         <mass value="0.0798"/>
-        <inertia ixx="0.002" ixy="0" ixz="0" iyy="0" iyz="0" izz="0" />
+        <inertia ixx="5.959597e-06" ixy="0" ixz="0" iyy="3.65197385e-05" iyz="0" izz="3.32798585e-05" />
       </inertial>
     </xacro:if>
@@ -119,5 +119,5 @@
         <origin xyz="-0.01 0 0" rpy="${mesh_offset_rpy}"/>
         <mass value="0.0798"/>
-        <inertia ixx="0.002" ixy="0" ixz="0" iyy="0" iyz="0" izz="0" />
+        <inertia ixx="5.959597e-06" ixy="0" ixz="0" iyy="3.65197385e-05" iyz="0" izz="3.32798585e-05" />
       </inertial>
     </xacro:if>

File: fetch_moveit_config/srdf/fetch_arm.xacro (robot description, xacro)
@@ -17,4 +17,13 @@
       <joint name="wrist_roll_joint" />
     </group>
+    <group_state group="arm" name="ready">
+      <joint name="shoulder_pan_joint" value="1.32"/>
+      <joint name="shoulder_lift_joint" value="0.7"/>
+      <joint name="upperarm_roll_joint" value="0.0"/>
+      <joint name="elbow_flex_joint" value="-2.0"/>
+      <joint name="forearm_roll_joint" value="0.0"/>
+      <joint name="wrist_flex_joint" value="-0.57"/>
+      <joint name="wrist_roll_joint" value="0.0"/>
+    </group_state>
     <!--DISABLE COLLISIONS: By default it is assumed that any link of the robot could potentially come into collision with any other link in the robot. This tag disables collision checking between a specified pair of links. -->
     <disable_collisions link1="base_link" link2="bellows_link" reason="Default" />
