Commit message: test successfully

File: fetch_description/urdf/fetch_arm.xacro (robot description, xacro)
@@ -127,5 +127,5 @@
     joint_damping="100.0"
     safety_limits="${safety_limits}"
-    safety_position_margin="${safety_position_margin}"
+    safety_position_margin="0.001"
     safety_k_position="${safety_k_position}"
     safety_k_velocity="${safety_k_velocity}"

File: fetch_moveit_config/srdf/fetch_arm.xacro (robot description, xacro)
@@ -8,5 +8,6 @@
     prefix:=fetch_
   ">
-    <group name="arm">
+    <group name="arm_with_torso">
+      <joint name="torso_lift_joint" />
       <joint name="shoulder_pan_joint" />
       <joint name="shoulder_lift_joint" />
@@ -17,5 +18,6 @@
       <joint name="wrist_roll_joint" />
     </group>
-    <group_state group="arm" name="ready">
+    <group_state group="arm_with_torso" name="ready">
+      <joint name="torso_lift_joint" value="0.38"/>
       <joint name="shoulder_pan_joint" value="1.32"/>
       <joint name="shoulder_lift_joint" value="0.7"/>
